File: Pipe-Hardware/pipe/pipe.kicad_pcb (KiCad board)
At the start: 2 copper layers, 100 x 100 mm, 16 parts, among them J1 Screw_Terminal_01x02, U1 ATmega32A-P, U2 MPU6050, U3 AT24C512B-PU25, U4 LLV, U5 AMS1117, U6 HC-5

Commit message: تعديل الإسطوانة
Parts:
- added D1: 1N4007, Diode_THT:D_DO-41_SOD81_P10.16mm_Horizontal, F.Cu at (126.2, 45.8)
- added J2: Screw_Terminal_01x02, TerminalBlock:TerminalBlock_MaiXu_MX126-5.0-02P_1x02_P5.00mm, F.Cu at (129.1, 38.6)
- added Q1: IRLZ44N, Package_TO_SOT_THT:TO-220-3_Vertical, F.Cu at (158.6, 50.2)
- added R4: 220, Resistor_THT:R_Axial_DIN0204_L3.6mm_D1.6mm_P5.08mm_Horizontal, F.Cu at (149.9, 50.2)
- added R5: 10k, Resistor_THT:R_Axial_DIN0204_L3.6mm_D1.6mm_P5.08mm_Horizontal, F.Cu at (164.6, 55.2)
Connections:
- U1 pad 40: unconnected-(U1-PA0-Pad40) -> Net-(U1-PA0)
Routing:
- net Net-(D1-A): track 0.00 -> 33.2 mm
- net Net-(D1-K): track 223.2 -> 251.5 mm
- net Net-(U1-PA0): track 0.00 -> 15.5 mm
- net Net-(Q1-G): track 0.00 -> 9.55 mm
