File: ROV-Hardware/ROV.kicad_sch (KiCad schematic)
At the start: 24 parts, among them J1 T-block, J2 Screw_Terminal_01x04, J3 Screw_Terminal_01x04, U2 LM7805, U3 ESP32-S3-DEVKITC-1-N8R2, U4 MPU6050, U5 ZK-BM1, U6 ZK-BM1, U7 ZK-BM1, U8 A4988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

Commit message: DC jack
Parts:
- added J4: Barrel_Jack_Switch, Connector_BarrelJack:BarrelJack_Horizontal, symbol Connector:Barrel_Jack_Switch
Connections:
- net GND: now also J4.2, J4.3
- net at C2.1, D3.2 (A), F2.1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: now also J4.1
Changed lines of the file:
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@@
 	)
 	(junction
+		(at 109.22 50.8)
+		(diameter 0)
+		(color 0 0 0 0)
+	)
+	(junction
 		(at 88.9 35.56)
 		(diameter 0)
@@
 	)
 	(junction
+		(at 109.22 35.56)
+		(diameter 0)
+		(color 0 0 0 0)
+	)
+	(junction
 		(at 72.39 50.8)
 		(diameter 0)
@@
 	)
 	(junction
+		(at 109.22 45.72)
+		(diameter 0)
+		(color 0 0 0 0)
+	)
+	(junction
 		(at 49.53 35.56)
 		(diameter 0)
@@
 	(wire
 		(pts
+			(xy 109.22 50.8) (xy 129.54 50.8)
+		)
+		(stroke
+			(width 0)
+			(type default)
+		)
+	)
+	(wire
+		(pts
 			(xy 88.9 50.8) (xy 91.44 50.8)
 		)
@@
 	(wire
 		(pts
-			(xy 91.44 50.8) (xy 97.79 50.8)
+			(xy 91.44 50.8) (xy 109.22 50.8)
 		)
 		(stroke
@@
 	(wire
 		(pts
+			(xy 109.22 43.18) (xy 109.22 45.72)
+		)
+		(stroke
+			(width 0)
+			(type default)
+		)
+	)
+	(wire
+		(pts
 			(xy 129.54 111.76) (xy 140.97 111.76)
 		)
@@
 	(wire
 		(pts
+			(xy 109.22 45.72) (xy 109.22 50.8)
+		)
+		(stroke
+			(width 0)
+			(type default)
+		)
+	)
+	(wire
+		(pts
 			(xy 186.69 33.02) (xy 186.69 35.56)
 		)
@@
 	(wire
 		(pts
+			(xy 109.22 35.56) (xy 133.35 35.56)
+		)
+		(stroke
+			(width 0)
+			(type default)
+		)
+	)
+	(wire
+		(pts
 			(xy 71.12 99.06) (xy 73.66 99.06)
 		)
@@
 	(wire
 		(pts
-			(xy 125.73 35.56) (xy 186.69 35.56)
+			(xy 152.4 35.56) (xy 186.69 35.56)
 		)
 		(stroke
@@
 	(wire
 		(pts
-			(xy 118.11 35.56) (xy 109.22 35.56)
+			(xy 144.78 35.56) (xy 140.97 35.56)
 		)
 		(stroke
@@
 	(wire
 		(pts
-			(xy 88.9 35.56) (xy 101.6 35.56)
+			(xy 88.9 35.56) (xy 109.22 35.56)
 		)
 		(stroke
@@
 	(wire
 		(pts
+			(xy 109.22 35.56) (xy 109.22 40.64)
+		)
+		(stroke
+			(width 0)
+			(type default)
+		)
+	)
+	(wire
+		(pts
 			(xy 49.53 60.96) (xy 49.53 35.56)
 		)
@@
 	(symbol
 		(lib_id "power:GNDREF")
-		(at 97.79 50.8 90)
+		(at 129.54 50.8 90)
 		(unit 1)
 		(exclude_from_sim no)
@@
 		(fields_autoplaced yes)
 		(property "Reference" "#PWR02"
-			(at 104.14 50.8 0)
+			(at 135.89 50.8 0)
 			(effects
 				(font
@@
 		)
 		(property "Value" "GNDREF"
-			(at 101.6 50.7999 90)
+			(at 133.35 50.7999 90)
 			(effects
 				(font
@@
 		)
 		(property "Footprint" ""
-			(at 97.79 50.8 0)
+			(at 129.54 50.8 0)
 			(effects
 				(font
@@
 		)
 		(property "Datasheet" ""
-			(at 97.79 50.8 0)
+			(at 129.54 50.8 0)
 			(effects
 				(font
@@
 		)
 		(property "Description" "Power symbol creates a global label with name \"GNDREF\" , reference supply ground"
-			(at 97.79 50.8 0)
+			(at 129.54 50.8 0)
 			(effects
 				(font
@@
 	)
 	(symbol
+		(lib_id "Connector:Barrel_Jack_Switch")
+		(at 116.84 43.18 0)
+		(mirror y)
+		(unit 1)
+		(exclude_from_sim no)
+		(in_bom yes)
+		(on_board yes)
+		(dnp no)
+		(fields_autoplaced yes)
+		(property "Reference" "J4"
+			(at 123.19 41.9099 0)
+			(effects
+				(font
+					(size 1.27 1.27)
+				)
+				(justify right)
+			)
+		)
+		(property "Value" "Barrel_Jack_Switch"
+			(at 123.19 44.4499 0)
+			(effects
+				(font
+					(size 1.27 1.27)
+				)
+				(justify right)
+			)
+		)
+		(property "Footprint" "Connector_BarrelJack:BarrelJack_Horizontal"
+			(at 115.57 44.196 0)
+			(effects
+				(font
+					(size 1.27 1.27)
+				)
+				(hide yes)
+			)
+		)
+		(property "Datasheet" "~"
+			(at 115.57 44.196 0)
+			(effects
+				(font
+					(size 1.27 1.27)
+				)
+				(hide yes)
+			)
+		)
+		(property "Description" "DC Barrel Jack with an internal switch"
+			(at 116.84 43.18 0)
+			(effects
+				(font
+					(size 1.27 1.27)
+				)
+				(hide yes)
+			)
+		)
+		(pin "1"
+		)
+		(pin "2"
+		)
+		(pin "3"
+		)
+		(instances
+			(project ""
+				(path "/df7a457f-e553-4b1a-9143-cdb39e42e745"
+					(reference "J4")
+					(unit 1)
+				)
+			)
+		)
+	)
+	(symbol
 		(lib_id "Device:Fuse")
 		(at 100.33 63.5 90)
@@
 	(symbol
 		(lib_id "Diode:1N5819")
-		(at 121.92 35.56 0)
+		(at 148.59 35.56 0)
 		(mirror y)
 		(unit 1)
@@
 		(dnp no)
 		(property "Reference" "D1"
-			(at 122.2375 29.21 0)
+			(at 148.9075 29.21 0)
 			(effects
 				(font
@@
 		)
 		(property "Value" "1N5819"
-			(at 122.2375 31.75 0)
+			(at 148.9075 31.75 0)
 			(effects
 				(font
@@
 		)
 		(property "Footprint" "Diode_THT:D_DO-41_SOD81_P10.16mm_Horizontal"
-			(at 121.92 40.005 0)
+			(at 148.59 40.005 0)
 			(effects
 				(font
@@
 		)
 		(property "Datasheet" "http://www.vishay.com/docs/88525/1n5817.pdf"
-			(at 121.92 35.56 0)
+			(at 148.59 35.56 0)
 			(effects
 				(font
@@
 		)
 		(property "Description" "40V 1A Schottky Barrier Rectifier Diode, DO-41"
-			(at 121.92 35.56 0)
+			(at 148.59 35.56 0)
 			(effects
 				(font
@@
 	(symbol
 		(lib_id "Device:Fuse")
-		(at 105.41 35.56 90)
+		(at 137.16 35.56 90)
 		(unit 1)
 		(exclude_from_sim no)
@@
 		(fields_autoplaced yes)
 		(property "Reference" "F2"
-			(at 105.41 29.21 90)
+			(at 137.16 29.21 90)
 			(effects
 				(font
@@
 		)
 		(property "Value" "fuse"
-			(at 105.41 31.75 90)
+			(at 137.16 31.75 90)
 			(effects
 				(font
@@
 		)
 		(property "Footprint" "Fuse:Fuseholder_Clip-5x20mm_Schurter_CQM_Inline_P20.60x5.00mm_D1.00mm_Horizontal"
-			(at 105.41 37.338 90)
+			(at 137.16 37.338 90)
 			(effects
 				(font
@@
 		)
 		(property "Datasheet" "~"
-			(at 105.41 35.56 0)
+			(at 137.16 35.56 0)
 			(effects
 				(font
@@
 		)
 		(property "Description" "Fuse"
-			(at 105.41 35.56 0)
+			(at 137.16 35.56 0)
 			(effects
 				(font

Commit message: fishs and starfishs
Parts:
- removed J4: Barrel_Jack_Switch, Connector_BarrelJack:BarrelJack_Horizontal, symbol Connector:Barrel_Jack_Switch
- added J4: T-block, TerminalBlock:TerminalBlock_MaiXu_MX126-5.0-02P_1x02_P5.00mm, symbol Connector:Screw_Terminal_01x02
- F3, F4, F5: footprint Fuse:Fuseholder_Clip-5x20mm_Schurter_CQM_Inline_P20.60x5.00mm_D1.00mm_Horizontal -> Fuse:Fuse_Blade_ATO_directSolder
Connections:
- net GND: now also J4.1 (Pin_1)
- net at C2.1, D3.2 (A), F2.1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: now also J4.2 (Pin_2)
Changed lines of the file:
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@@
-	)
-	(junction
-		(at 109.22 50.8)
-		(diameter 0)
-		(color 0 0 0 0)
 	)
 	(junction
@@
 	)
 	(junction
-		(at 109.22 35.56)
-		(diameter 0)
-		(color 0 0 0 0)
-	)
-	(junction
 		(at 72.39 50.8)
 		(diameter 0)
@@
 	)
 	(junction
+		(at 100.33 50.8)
+		(diameter 0)
+		(color 0 0 0 0)
+	)
+	(junction
 		(at 91.44 50.8)
 		(diameter 0)
@@
 	)
 	(junction
-		(at 109.22 45.72)
+		(at 49.53 35.56)
 		(diameter 0)
 		(color 0 0 0 0)
 	)
 	(junction
-		(at 49.53 35.56)
+		(at 100.33 35.56)
 		(diameter 0)
 		(color 0 0 0 0)
@@
 	(wire
 		(pts
-			(xy 109.22 50.8) (xy 129.54 50.8)
-		)
-		(stroke
-			(width 0)
-			(type default)
-		)
-	)
-	(wire
-		(pts
 			(xy 88.9 50.8) (xy 91.44 50.8)
 		)
@@
 	(wire
 		(pts
-			(xy 91.44 50.8) (xy 109.22 50.8)
+			(xy 91.44 50.8) (xy 100.33 50.8)
 		)
 		(stroke
@@
 	(wire
 		(pts
-			(xy 109.22 43.18) (xy 109.22 45.72)
-		)
-		(stroke
-			(width 0)
-			(type default)
-		)
-	)
-	(wire
-		(pts
 			(xy 129.54 111.76) (xy 140.97 111.76)
 		)
@@
 	(wire
 		(pts
+			(xy 100.33 35.56) (xy 100.33 41.91)
+		)
+		(stroke
+			(width 0)
+			(type default)
+		)
+	)
+	(wire
+		(pts
 			(xy 208.28 71.12) (xy 208.28 85.09)
 		)
@@
 	(wire
 		(pts
-			(xy 109.22 45.72) (xy 109.22 50.8)
-		)
-		(stroke
-			(width 0)
-			(type default)
-		)
-	)
-	(wire
-		(pts
 			(xy 186.69 33.02) (xy 186.69 35.56)
 		)
@@
 	(wire
 		(pts
+			(xy 100.33 35.56) (xy 133.35 35.56)
+		)
+		(stroke
+			(width 0)
+			(type default)
+		)
+	)
+	(wire
+		(pts
 			(xy 58.42 50.8) (xy 72.39 50.8)
 		)
@@
 	(wire
 		(pts
-			(xy 109.22 35.56) (xy 133.35 35.56)
+			(xy 88.9 35.56) (xy 100.33 35.56)
 		)
 		(stroke
@@
 	(wire
 		(pts
+			(xy 100.33 50.8) (xy 129.54 50.8)
+		)
+		(stroke
+			(width 0)
+			(type default)
+		)
+	)
+	(wire
+		(pts
+			(xy 100.33 44.45) (xy 100.33 50.8)
+		)
+		(stroke
+			(width 0)
+			(type default)
+		)
+	)
+	(wire
+		(pts
 			(xy 134.62 48.26) (xy 134.62 76.2)
 		)
@@
 	(wire
 		(pts
-			(xy 88.9 35.56) (xy 109.22 35.56)
-		)
-		(stroke
-			(width 0)
-			(type default)
-		)
-	)
-	(wire
-		(pts
 			(xy 91.44 58.42) (xy 91.44 50.8)
 		)
@@
 		(pts
 			(xy 82.55 35.56) (xy 88.9 35.56)
-		)
-		(stroke
-			(width 0)
-			(type default)
-		)
-	)
-	(wire
-		(pts
-			(xy 109.22 35.56) (xy 109.22 40.64)
 		)
 		(stroke
@@
 	)
 	(symbol
+		(lib_id "Connector:Screw_Terminal_01x02")
+		(at 105.41 44.45 0)
+		(mirror x)
+		(unit 1)
+		(exclude_from_sim no)
+		(in_bom yes)
+		(on_board yes)
+		(dnp no)
+		(property "Reference" "J4"
+			(at 105.41 35.56 0)
+			(effects
+				(font
+					(size 1.27 1.27)
+				)
+				(hide yes)
+			)
+		)
+		(property "Value" "T-block"
+			(at 105.41 38.1 0)
+			(effects
+				(font
+					(size 1.27 1.27)
+				)
+				(hide yes)
+			)
+		)
+		(property "Footprint" "TerminalBlock:TerminalBlock_MaiXu_MX126-5.0-02P_1x02_P5.00mm"
+			(at 105.41 44.45 0)
+			(effects
+				(font
+					(size 1.27 1.27)
+				)
+				(hide yes)
+			)
+		)
+		(property "Datasheet" "~"
+			(at 105.41 44.45 0)
+			(effects
+				(font
+					(size 1.27 1.27)
+				)
+				(hide yes)
+			)
+		)
+		(property "Description" "Generic screw terminal, single row, 01x02, script generated (kicad-library-utils/schlib/autogen/connector/)"
+			(at 105.41 44.45 0)
+			(effects
+				(font
+					(size 1.27 1.27)
+				)
+				(hide yes)
+			)
+		)
+		(pin "1"
+		)
+		(pin "2"
+		)
+		(instances
+			(project "ROV"
+				(path "/df7a457f-e553-4b1a-9143-cdb39e42e745"
+					(reference "J4")
+					(unit 1)
+				)
+			)
+		)
+	)
+	(symbol
 		(lib_id "MPU6050:GY-MS5837")
 		(at 220.98 72.39 0)
@@
 			)
 		)
-		(property "Footprint" "Fuse:Fuseholder_Clip-5x20mm_Schurter_CQM_Inline_P20.60x5.00mm_D1.00mm_Horizontal"
+		(property "Footprint" "Fuse:Fuse_Blade_ATO_directSolder"
 			(at 100.33 67.818 90)
 			(effects
@@
 	)
 	(symbol
-		(lib_id "Connector:Barrel_Jack_Switch")
-		(at 116.84 43.18 0)
-		(mirror y)
-		(unit 1)
-		(exclude_from_sim no)
-		(in_bom yes)
-		(on_board yes)
-		(dnp no)
-		(fields_autoplaced yes)
-		(property "Reference" "J4"
-			(at 123.19 41.9099 0)
-			(effects
-				(font
-					(size 1.27 1.27)
-				)
-				(justify right)
-			)
-		)
-		(property "Value" "Barrel_Jack_Switch"
-			(at 123.19 44.4499 0)
-			(effects
-				(font
-					(size 1.27 1.27)
-				)
-				(justify right)
-			)
-		)
-		(property "Footprint" "Connector_BarrelJack:BarrelJack_Horizontal"
-			(at 115.57 44.196 0)
-			(effects
-				(font
-					(size 1.27 1.27)
-				)
-				(hide yes)
-			)
-		)
-		(property "Datasheet" "~"
-			(at 115.57 44.196 0)
-			(effects
-				(font
-					(size 1.27 1.27)
-				)
-				(hide yes)
-			)
-		)
-		(property "Description" "DC Barrel Jack with an internal switch"
-			(at 116.84 43.18 0)
-			(effects
-				(font
-					(size 1.27 1.27)
-				)
-				(hide yes)
-			)
-		)
-		(pin "1"
-		)
-		(pin "2"
-		)
-		(pin "3"
-		)
-		(instances
-			(project ""
-				(path "/df7a457f-e553-4b1a-9143-cdb39e42e745"
-					(reference "J4")
-					(unit 1)
-				)
-			)
-		)
-	)
-	(symbol
 		(lib_id "Device:Fuse")
 		(at 100.33 63.5 90)
@@
 			)
 		)
-		(property "Footprint" "Fuse:Fuseholder_Clip-5x20mm_Schurter_CQM_Inline_P20.60x5.00mm_D1.00mm_Horizontal"
+		(property "Footprint" "Fuse:Fuse_Blade_ATO_directSolder"
 			(at 100.33 65.278 90)
 			(effects
@@
 			)
 		)
-		(property "Footprint" "Fuse:Fuseholder_Clip-5x20mm_Schurter_CQM_Inline_P20.60x5.00mm_D1.00mm_Horizontal"
+		(property "Footprint" "Fuse:Fuse_Blade_ATO_directSolder"
 			(at 100.33 62.738 90)
 			(effects

Commit message: وجع القلب
Other:
- moved on the sheet: U10
Changed lines of the file:
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@@
+	(wire
+		(pts
+			(xy 92.71 88.9) (xy 91.44 88.9)
+		)
+		(stroke
+			(width 0)
+			(type default)
+		)
+	)
 	(wire
 		(pts
@@
 	(wire
 		(pts
+			(xy 222.25 60.96) (xy 220.98 60.96)
+		)
+		(stroke
+			(width 0)
+			(type default)
+		)
+	)
+	(wire
+		(pts
 			(xy 73.66 93.98) (xy 73.66 96.52)
 		)
@@
 	(wire
 		(pts
-			(xy 208.28 58.42) (xy 220.98 58.42)
+			(xy 208.28 58.42) (xy 222.25 58.42)
 		)
 		(stroke
@@
 	(wire
 		(pts
-			(xy 220.98 55.88) (xy 220.98 48.26)
+			(xy 215.9 55.88) (xy 215.9 48.26)
 		)
 		(stroke
@@
 	(wire
 		(pts
+			(xy 92.71 93.98) (xy 91.44 93.98)
+		)
+		(stroke
+			(width 0)
+			(type default)
+		)
+	)
+	(wire
+		(pts
 			(xy 106.68 109.22) (xy 71.12 109.22)
 		)
@@
 	(wire
 		(pts
+			(xy 215.9 55.88) (xy 222.25 55.88)
+		)
+		(stroke
+			(width 0)
+			(type default)
+		)
+	)
+	(wire
+		(pts
 			(xy 91.44 63.5) (xy 96.52 63.5)
 		)
@@
 	(wire
 		(pts
+			(xy 92.71 91.44) (xy 91.44 91.44)
+		)
+		(stroke
+			(width 0)
+			(type default)
+		)
+	)
+	(wire
+		(pts
+			(xy 92.71 96.52) (xy 91.44 96.52)
+		)
+		(stroke
+			(width 0)
+			(type default)
+		)
+	)
+	(wire
+		(pts
 			(xy 129.54 116.84) (xy 137.16 116.84)
 		)
@@
 	(wire
 		(pts
-			(xy 220.98 48.26) (xy 134.62 48.26)
+			(xy 215.9 48.26) (xy 134.62 48.26)
 		)
 		(stroke
@@
 		(pts
 			(xy 49.53 60.96) (xy 91.44 60.96)
+		)
+		(stroke
+			(width 0)
+			(type default)
+		)
+	)
+	(wire
+		(pts
+			(xy 208.28 107.95) (xy 208.28 105.41)
 		)
 		(stroke
@@
 	(symbol
 		(lib_id "power:GNDREF")
-		(at 208.28 105.41 0)
+		(at 208.28 107.95 0)
 		(unit 1)
 		(exclude_from_sim no)
@@
 		(dnp no)
 		(property "Reference" "#PWR04"
-			(at 208.28 111.76 0)
+			(at 208.28 114.3 0)
 			(effects
 				(font
@@
 		)
 		(property "Value" "GNDREF"
-			(at 214.122 106.934 0)
+			(at 214.122 109.474 0)
 			(effects
 				(font
@@
 		)
 		(property "Footprint" ""
-			(at 208.28 105.41 0)
+			(at 208.28 107.95 0)
 			(effects
 				(font
@@
 		)
 		(property "Datasheet" ""
-			(at 208.28 105.41 0)
+			(at 208.28 107.95 0)
 			(effects
 				(font
@@
 		)
 		(property "Description" "Power symbol creates a global label with name \"GNDREF\" , reference supply ground"
-			(at 208.28 105.41 0)
+			(at 208.28 107.95 0)
 			(effects
 				(font
@@
 	(symbol
 		(lib_id "Connector:Screw_Terminal_01x04")
-		(at 96.52 91.44 0)
+		(at 97.79 91.44 0)
 		(unit 1)
 		(exclude_from_sim no)
@@
 		(fields_autoplaced yes)
 		(property "Reference" "J3"
-			(at 99.06 91.4399 0)
+			(at 100.33 91.4399 0)
 			(effects
 				(font
@@
 		)
 		(property "Value" "Screw_Terminal_01x04"
-			(at 99.06 93.9799 0)
+			(at 100.33 93.9799 0)
 			(effects
 				(font
@@
 		)
 		(property "Footprint" "TerminalBlock:TerminalBlock_MaiXu_MX126-5.0-04P_1x04_P5.00mm"
-			(at 96.52 91.44 0)
+			(at 97.79 91.44 0)
 			(effects
 				(font
@@
 		)
 		(property "Datasheet" "~"
-			(at 96.52 91.44 0)
+			(at 97.79 91.44 0)
 			(effects
 				(font
@@
 		)
 		(property "Description" "Generic screw terminal, single row, 01x04, script generated (kicad-library-utils/schlib/autogen/connector/)"
-			(at 96.52 91.44 0)
+			(at 97.79 91.44 0)
 			(effects
 				(font
@@
 	(symbol
 		(lib_id "MPU6050:water")
-		(at 226.06 58.42 0)
+		(at 227.33 58.42 0)
 		(unit 1)
 		(exclude_from_sim no)
@@
 		(fields_autoplaced yes)
 		(property "Reference" "U10"
-			(at 229.87 57.1499 0)
+			(at 231.14 57.1499 0)
 			(effects
 				(font
@@
 		)
 		(property "Value" "~"
-			(at 229.87 59.6899 0)
+			(at 231.14 59.6899 0)
 			(effects
 				(font
@@
 		)
 		(property "Footprint" "Connector_PinHeader_2.54mm:PinHeader_1x03_P2.54mm_Vertical"
-			(at 226.06 58.42 0)
+			(at 227.33 58.42 0)
 			(effects
 				(font
@@
 		)
 		(property "Datasheet" ""
-			(at 226.06 58.42 0)
+			(at 227.33 58.42 0)
 			(effects
 				(font
@@
 		)
 		(property "Description" ""
-			(at 226.06 58.42 0)
-			(effects
-				(font
+			(at 227.33 58.42 0)
+			(effects
+				(font
