File: ROV-Hardware/ROV.kicad_sch (KiCad schematic)
At the start: 25 parts, among them J1 T-block, J2 Screw_Terminal_01x04, J3 Screw_Terminal_01x04, J4 T-block, U2 LM7805, U3 ESP32-S3-DEVKITC-1-N8R2, U4 MPU6050, U5 ZK-BM1, U6 ZK-BM1, U7 ZK-BM1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

Commit message: pipe 2
Parts:
- removed U2: LM7805, Package_TO_SOT_THT:TO-220-3_Vertical, symbol Regulator_Linear:LM7805_TO220
- added U1: LM2596, Connector_PinHeader_2.54mm:PinHeader_1x04_P2.54mm_Vertical, symbol MPU6050:LM2596
Connections:
- net GND: now also C1.2, U1.2 (IN-), U1.3 (OUT-); no longer C1.1
- net at D2.2 (A), F1.2, F3.1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: now also C1.1, U1.1 (IN+); no longer C1.2
- net at C2.1, D3.2 (A), F2.1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: now also U1.4 (OUT+)
