File: ROV-Hardware/ROV.kicad_sch (KiCad schematic)
At the start: 27 parts, among them J1 T-block, J2 T-block, J3 Screw_Terminal_01x04, J4 T-block, J5 T-block, J6 T-block, U1 LM2596, U3 ESP32-S3-DEVKITC-1-N8R2, U4 MPU6050, U5 ZK-BM1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

Commit message: refresh
Parts:
- J2, J5, J6: footprint Connector_AMASS:AMASS_XT60-F_1x02_P7.20mm_Vertical -> TerminalBlock:TerminalBlock_MaiXu_MX126-5.0-02P_1x02_P5.00mm
Changed lines of the file:
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@@
 			)
 		)
-		(property "Footprint" "Connector_AMASS:AMASS_XT60-F_1x02_P7.20mm_Vertical"
+		(property "Footprint" "TerminalBlock:TerminalBlock_MaiXu_MX126-5.0-02P_1x02_P5.00mm"
 			(at 88.9 60.96 0)
 			(effects
@@
 			)
 		)
-		(property "Footprint" "Connector_AMASS:AMASS_XT60-F_1x02_P7.20mm_Vertical"
+		(property "Footprint" "TerminalBlock:TerminalBlock_MaiXu_MX126-5.0-02P_1x02_P5.00mm"
 			(at 88.9 71.12 0)
 			(effects
@@
 			)
 		)
-		(property "Footprint" "Connector_AMASS:AMASS_XT60-F_1x02_P7.20mm_Vertical"
+		(property "Footprint" "TerminalBlock:TerminalBlock_MaiXu_MX126-5.0-02P_1x02_P5.00mm"
 			(at 88.9 66.04 0)
 			(effects
