File: ROV-Hardware/ROV.kicad_pcb (KiCad board)
At the start: 2 copper layers, 130 x 90 mm, 29 parts, among them J1 T-block, J2 Screw_Terminal_01x04, J3 Screw_Terminal_01x04, J4 T-block, U1 LM2596, U3 ESP32-S3-DEVKITC-1-N8R2, U4 MPU6050, U5 ZK-BM1, U6 ZK-BM1, U7 ZK-BM1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

Commit message: refresh
Parts:
- added G***: LOGO, logo:logo5, B.Cu at (139.6, 114.3)
Routing:
- net +5V: track 31.1 -> 62.2 mm

Commit message: refresh
Routing:
- net Net-(D1-A): track 26.7 -> 57.2 mm
Changed lines of the file:
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@@
 		(tenting front back)
 		(pcbplotparams
-			(layerselection 0x00000000_00000000_55555555_55555551)
+			(layerselection 0x00000000_00000000_55555555_55555555)
 			(plot_on_all_layers_selection 0x00000000_00000000_00000000_00000000)
 			(disableapertmacros no)
@@
 			(dxfimperialunits yes)
 			(dxfusepcbnewfont yes)
-			(psnegative no)
+			(psnegative yes)
 			(psa4output no)
 			(plot_black_and_white yes)
@@
 			(subtractmaskfromsilk no)
 			(outputformat 4)
-			(mirror no)
+			(mirror yes)
 			(drillshape 2)
 			(scaleselection 1)
@@
 	)
 	(segment
+		(start 162.33 67.315)
+		(end 160.575 65.56)
+		(width 2)
+		(layer "F.Cu")
+		(net 16)
+	)
+	(segment
+		(start 160.575 65.56)
+		(end 157.33 62.315)
+		(width 2)
+		(layer "F.Cu")
+		(net 16)
+	)
+	(segment
+		(start 163.36 67.315)
+		(end 162.33 67.315)
+		(width 2)
+		(layer "F.Cu")
+		(net 16)
+	)
+	(segment
+		(start 157.33 62.315)
+		(end 158.36 62.315)
+		(width 2)
+		(layer "F.Cu")
+		(net 16)
+	)
+	(segment
+		(start 157.33 65.56)
+		(end 157.33 62.315)
+		(width 2)
+		(layer "F.Cu")
+		(net 16)
+	)
+	(segment
+		(start 157.33 65.56)
+		(end 160.575 65.56)
+		(width 2)
+		(layer "F.Cu")
+		(net 16)
+	)
+	(segment
+		(start 157.33 67.315)
+		(end 157.33 65.56)
+		(width 2)
+		(layer "F.Cu")
+		(net 16)
+	)
+	(segment
+		(start 157.33 67.315)
+		(end 163.36 67.315)
+		(width 2)
+		(layer "F.Cu")
+		(net 16)
+	)
+	(segment
+		(start 158.36 62.315)
+		(end 163.36 67.315)
+		(width 2)
+		(layer "F.Cu")
+		(net 16)
+	)
+	(segment

Commit message: refresh
Parts:
- added J5: T-block, TerminalBlock:TerminalBlock_MaiXu_MX126-5.0-02P_1x02_P5.00mm, F.Cu at (88.0, 83.3)
- added J6: T-block, TerminalBlock:TerminalBlock_MaiXu_MX126-5.0-02P_1x02_P5.00mm, F.Cu at (88.0, 70.2)
- J2: value Screw_Terminal_01x04 -> T-block; footprint TerminalBlock:TerminalBlock_MaiXu_MX126-5.0-04P_1x04_P5.00mm -> TerminalBlock:TerminalBlock_MaiXu_MX126-5.0-02P_1x02_P5.00mm
- moved F5 32.1 mm to (108.0, 65.2)
- moved J1 16.3 mm to (127.8, 60.2), turned to 180 degrees
- moved J2 13.8 mm to (88.0, 96.3), turned to 90 degrees
- moved F4 11.9 mm to (108.0, 78.3)
- moved F3 8.45 mm to (108.0, 91.4)
- moved F1 1.03 mm to (120.6, 70.8)
- moved R1 0.72 mm to (139.4, 82.9)
- moved D2 0.58 mm to (131.5, 82.9)
Connections:
- F4 pad 2: Net-(J2-Pin_3) -> Net-(J5-Pin_2)
- F5 pad 2: Net-(J2-Pin_4) -> Net-(J6-Pin_2)
Routing:
- net Net-(D2-A): track 286.6 -> 793.1 mm
- net Net-(J2-Pin_4): track 48.2 -> 0.00 mm
- net Net-(J2-Pin_3): track 39.0 -> 0.00 mm
- net Net-(J2-Pin_2): track 54.3 -> 21.6 mm
- net Net-(J6-Pin_2): track 0.00 -> 21.5 mm
- net Net-(J5-Pin_2): track 0.00 -> 21.5 mm
- net +12V: track 18.2 -> 21.2 mm
- net Net-(J3-Pin_1): track 18.7 -> 19.3 mm

Commit message: refresh
Routing:
- net Net-(U10-S): track 66.7 -> 65.6 mm
Changed lines of the file:
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@@
 	)
 	(segment
-		(start 179.794466 137.260534)
-		(end 188.915282 128.139718)
+		(start 199.23 124.625)
+		(end 198.643203 124.625)
+		(width 2)
+		(layer "F.Cu")
+		(net 56)
+	)
+	(segment
+		(start 184.501067 130.482865)
+		(end 182.116796 132.867136)
 		(width 2)
 		(layer "F.Cu")
@@
 	(segment
 		(start 147.97 138.725)
-		(end 176.258932 138.725)
+		(end 167.974661 138.725)
 		(width 2)
 		(layer "F.Cu")
 		(net 56)
 	)
-	(segment
-		(start 197.400563 124.625)
-		(end 199.23 124.625)
+	(arc
+		(start 182.116796 132.867136)
+		(mid 175.628329 137.202591)
+		(end 167.974661 138.725)
 		(width 2)
 		(layer "F.Cu")
@@
 	)
 	(arc
-		(start 188.915282 128.139718)
-		(mid 192.808362 125.538445)
-		(end 197.400563 124.625)
-		(width 2)
-		(layer "F.Cu")
-		(net 56)
-	)
-	(arc
-		(start 179.794466 137.260534)
-		(mid 178.172349 138.344398)
-		(end 176.258932 138.725)
+		(start 184.501067 130.482865)
+		(mid 190.989534 126.14741)
+		(end 198.643203 124.625)
 		(width 2)
 		(layer "F.Cu")
@@
 		(polygon
 			(pts
-				(xy 312.44 -85.575) (xy -10.47 -14.375) (xy -0.12 220.355) (xy 165.47 220.355) (xy 360.39 221.725)
+				(xy 329.66 -47.22) (xy -10.47 -14.375) (xy -0.12 220.355) (xy 165.47 220.355) (xy 360.39 221.725)
 			)
 		)
